File: 2.Satellite/1.Hardware/Boards/avionics-solarpanels/Solar-Panel-X- (4L)/Solar-Panel-X-.kicad_pcb (KiCad board)
At the start: 4 copper layers, 48.4 x 48.4 mm, 81 parts, among them J1 FTS-105-01-X-DV-A, Q1 NX3008NBKS, Q2 MBT2222ADW1T1, Q3 NX3008NBKS, Q4 MBT2222ADW1T1, U1 BQ25570RGRR, U2 OPT3001, U3 MAX40200AUK

Commit message: update HW
Other:
- board text removed: "JLCJLCJLCJLC"
Changed lines of the file:
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@@
         (effects (font (size 1 1) (thickness 0.15)))
     )
-    (fp_rect (start -4.4902 -3.0176) (end -3.7902 0.0824)
-      (stroke (width 0.12) (type solid)) (fill solid) (layer "F.SilkS"))
     (fp_rect (start -2.5902 -1.1176) (end -5.6902 -1.8176)
       (stroke (width 0.12) (type solid)) (fill solid) (layer "F.SilkS"))
@@
     (effects (font (size 0.508 0.508) (thickness 0.1016)))
   )
-  (gr_text "JLCJLCJLCJLC" (at 94.6 79.7) (layer "F.SilkS")
-    (effects (font (size 0.635 0.635) (thickness 0.1016)))
-  )
   (gr_text "(4L)" (at 110.35 84.65) (layer "F.SilkS")
