File: 2.Satellite/1.Hardware/Boards/avionics-solarpanels/Solar-Panel-X- (4L)/BusProtection.kicad_sch (KiCad schematic)
At the start: 18 parts, among them Q1 NX3008NBKS, Q2 MBT2222ADW1T1, Q3 NX3008NBKS, Q4 MBT2222ADW1T1

Commit message: update HW
Other:
- note added: "Solar Panel Board X-"
- note removed: "Solar Panel Board X"
Changed lines of the file:
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@@
     (stroke (width 0) (type default))
   )
-  (text "Solar Panel Board X" (at 200.533 176.149 0)
+  (text "Solar Panel Board X-" (at 200.533 176.149 0)
     (effects (font (size 3.81 3.81) (thickness 0.762) bold) (justify left bottom))
   )
@@
     (pin "2")
     (instances
-      (project "Solar-Panel-X"
+      (project "Solar-Panel-X-"
         (path "/b5352a33-563a-4ffe-a231-2e68fb54afa3"
           (reference "R19") (unit 1)
@@
     (pin "1")
     (instances
-      (project "Solar-Panel-X"
+      (project "Solar-Panel-X-"
         (path "/b5352a33-563a-4ffe-a231-2e68fb54afa3"
           (reference "#PWR0111") (unit 1)
@@
     (pin "5")
     (instances
-      (project "Solar-Panel-X"
+      (project "Solar-Panel-X-"
         (path "/b5352a33-563a-4ffe-a231-2e68fb54afa3"
           (reference "Q2") (unit 2)
@@
     (pin "2")
     (instances
-      (project "Solar-Panel-X"
+      (project "Solar-Panel-X-"
         (path "/b5352a33-563a-4ffe-a231-2e68fb54afa3"
           (reference "R27") (unit 1)
@@
     (pin "1")
     (instances
-      (project "Solar-Panel-X"
+      (project "Solar-Panel-X-"
         (path "/b5352a33-563a-4ffe-a231-2e68fb54afa3"
           (reference "#PWR0108") (unit 1)
@@
     (pin "5")
     (instances
-      (project "Solar-Panel-X"
+      (project "Solar-Panel-X-"
         (path "/b5352a33-563a-4ffe-a231-2e68fb54afa3"
           (reference "Q2") (unit 1)
@@
     (pin "2")
     (instances
-      (project "Solar-Panel-X"
+      (project "Solar-Panel-X-"
         (path "/b5352a33-563a-4ffe-a231-2e68fb54afa3"
           (reference "R25") (unit 1)
@@
     (pin "5")
     (instances
-      (project "Solar-Panel-X"
+      (project "Solar-Panel-X-"
         (path "/b5352a33-563a-4ffe-a231-2e68fb54afa3"
           (reference "Q4") (unit 2)
@@
     (pin "1")
     (instances
-      (project "Solar-Panel-X"
+      (project "Solar-Panel-X-"
         (path "/b5352a33-563a-4ffe-a231-2e68fb54afa3"
           (reference "#PWR0107") (unit 1)
@@
     (pin "2")
     (instances
-      (project "Solar-Panel-X"
+      (project "Solar-Panel-X-"
         (path "/b5352a33-563a-4ffe-a231-2e68fb54afa3"
           (reference "R23") (unit 1)
@@
     (pin "2")
     (instances
-      (project "Solar-Panel-X"
+      (project "Solar-Panel-X-"
         (path "/b5352a33-563a-4ffe-a231-2e68fb54afa3"
           (reference "R30") (unit 1)
@@
     (pin "2")
     (instances
-      (project "Solar-Panel-X"
+      (project "Solar-Panel-X-"
         (path "/b5352a33-563a-4ffe-a231-2e68fb54afa3"
           (reference "C13") (unit 1)
@@
     (pin "5")
     (instances
-      (project "Solar-Panel-X"
+      (project "Solar-Panel-X-"
         (path "/b5352a33-563a-4ffe-a231-2e68fb54afa3"
           (reference "Q3") (unit 1)
@@
     (pin "2")
     (instances
-      (project "Solar-Panel-X"
+      (project "Solar-Panel-X-"
         (path "/b5352a33-563a-4ffe-a231-2e68fb54afa3"
           (reference "R24") (unit 1)
@@
     (pin "1")
     (instances
-      (project "Solar-Panel-X"
+      (project "Solar-Panel-X-"
         (path "/b5352a33-563a-4ffe-a231-2e68fb54afa3"
           (reference "#PWR0110") (unit 1)
@@
     (pin "5")
     (instances
-      (project "Solar-Panel-X"
+      (project "Solar-Panel-X-"
         (path "/b5352a33-563a-4ffe-a231-2e68fb54afa3"
           (reference "Q1") (unit 1)
@@
     (pin "2")
     (instances
-      (project "Solar-Panel-X"
+      (project "Solar-Panel-X-"
         (path "/b5352a33-563a-4ffe-a231-2e68fb54afa3"
           (reference "R20") (unit 1)
@@
     (pin "2")
     (instances
-      (project "Solar-Panel-X"
+      (project "Solar-Panel-X-"
         (path "/b5352a33-563a-4ffe-a231-2e68fb54afa3"
           (reference "R28") (unit 1)
@@
     (pin "5")
     (instances
-      (project "Solar-Panel-X"
+      (project "Solar-Panel-X-"
         (path "/b5352a33-563a-4ffe-a231-2e68fb54afa3"
           (reference "Q1") (unit 2)
@@
     (pin "2")
     (instances
-      (project "Solar-Panel-X"
+      (project "Solar-Panel-X-"
         (path "/b5352a33-563a-4ffe-a231-2e68fb54afa3"
           (reference "R21") (unit 1)
@@
     (pin "2")
     (instances
-      (project "Solar-Panel-X"
+      (project "Solar-Panel-X-"
         (path "/b5352a33-563a-4ffe-a231-2e68fb54afa3"
           (reference "C12") (unit 1)
@@
     (pin "1")
     (instances
-      (project "Solar-Panel-X"
+      (project "Solar-Panel-X-"
         (path "/b5352a33-563a-4ffe-a231-2e68fb54afa3"
           (reference "#PWR0109") (unit 1)
@@
     (pin "2")
     (instances
-      (project "Solar-Panel-X"
+      (project "Solar-Panel-X-"
         (path "/b5352a33-563a-4ffe-a231-2e68fb54afa3"
           (reference "R26") (unit 1)
@@
     (pin "5")
     (instances
-      (project "Solar-Panel-X"
+      (project "Solar-Panel-X-"
         (path "/b5352a33-563a-4ffe-a231-2e68fb54afa3"
           (reference "Q4") (unit 1)
@@
     (pin "5")
     (instances
-      (project "Solar-Panel-X"
+      (project "Solar-Panel-X-"
         (path "/b5352a33-563a-4ffe-a231-2e68fb54afa3"
           (reference "Q3") (unit 2)
@@
     (pin "1")
     (instances
-      (project "Solar-Panel-X"
+      (project "Solar-Panel-X-"
         (path "/b5352a33-563a-4ffe-a231-2e68fb54afa3"
           (reference "#PWR0106") (unit 1)
@@
     (pin "2")
     (instances
-      (project "Solar-Panel-X"
+      (project "Solar-Panel-X-"
         (path "/b5352a33-563a-4ffe-a231-2e68fb54afa3"
           (reference "R22") (unit 1)
@@
     (pin "2")
     (instances
-      (project "Solar-Panel-X"
+      (project "Solar-Panel-X-"
         (path "/b5352a33-563a-4ffe-a231-2e68fb54afa3"
           (reference "R29") (unit 1)

Commit message: update BOM
Parts:
- C12, C13: Manufacturer_Name (none) -> KYOCERA AVX; Manufacturer_Part_Number (none) -> 06031C103K4T4A; Package/Footprint (none) -> 0603; Website (none) -> https://www.digikey.pt/pt/products/detail/kyocera-avx/KAM15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
- Q1, Q3: Manufacturer_Part_Number NX3008NBKS -> NX3008NBKS,115; Package/Footprint (none) -> 6-TSSOP; Website (none) -> https://www.digikey.pt/pt/products/detail/nexperia-usa-inc/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
- Q2, Q4: Flight MBT2222ADW1T1G -> (none); Manufacturer_Name ON Semiconductor -> onsemi; Package/Footprint (none) -> SOT-363; Proto MBT2222ADW1T1G -> (none); Website (none) -> https://www.digikey.pt/pt/products/detail/onsemi/MBT2222ADW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
- R21, R26: Manufacturer_Name (none) -> Stackpole Electronics Inc; Manufacturer_Part_Number (none) -> RMCF0603FT680R; Package/Footprint (none) -> 0603; Website (none) -> https://www.digikey.pt/pt/products/detail/stackpole-electro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
- R22, R27: Manufacturer_Name (none) -> Stackpole Electronics Inc; Manufacturer_Part_Number (none) -> RNCF0603DTE100K; Package/Footprint (none) -> 0603; Website (none) -> https://www.digikey.pt/pt/products/detail/stackpole-electro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
- R23, R24, R28, R29: Manufacturer_Name (none) -> Stackpole Electronics Inc; Manufacturer_Part_Number (none) -> RNCF0603BTE10K0; Package/Footprint (none) -> 0603; Website (none) -> https://www.digikey.pt/pt/products/detail/stackpole-electro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
- R25, R30: Manufacturer_Name (none) -> Stackpole Electronics Inc; Manufacturer_Part_Number (none) -> RMCF0603FT200K; Package/Footprint (none) -> 0603; Website (none) -> https://www.digikey.pt/pt/products/detail/stackpole-electro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
Other:
- note added: "Solar Panel Board X+"
- note removed: "Solar Panel Board X-"
