File: 2.Satellite/1.Hardware/Boards/avionics-batteryboard/batteryboard-bottom/Bus Protection.kicad_sch (KiCad schematic)
At the start: 18 parts, among them Q1 NX3008NBKS, Q2 MBT2222ADW1T1, Q3 NX3008NBKS, Q4 MBT2222ADW1T1

Commit message: update BOM
Parts:
- C12, C13: Manufacturer_Name (none) -> KYOCERA AVX; Manufacturer_Part_Number (none) -> 06031C103K4T4A; Package/Footprint (none) -> 0603; Website (none) -> https://www.digikey.pt/pt/products/detail/kyocera-avx/KAM15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
- Q1: Flight BSS138DWQ-7 -> (none); LCSC Part# C396098 -> (none); Package/Footprint (none) -> 6-TSSOP
- Q2, Q4: Flight MBT2222ADW1T1G -> (none); LCSC Part# C157366 -> (none); Manufacturer_Name ON Semiconductor -> onsemi; Package/Footprint (none) -> SOT-363; Proto MBT2222ADW1T1G -> (none)
- Q3: LCSC Part# C396098 -> (none); Package/Footprint (none) -> 6-TSSOP
- R19, R20: Manufacturer_Name (none) -> Stackpole Electronics Inc; Manufacturer_Part_Number (none) -> RMCF0603ZT0R00; Package/Footprint (none) -> 0603; Website (none) -> https://www.digikey.pt/pt/products/detail/stackpole-electro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
- R21, R26: Manufacturer_Name (none) -> Stackpole Electronics Inc; Manufacturer_Part_Number (none) -> RMCF0603FT680R; Package/Footprint (none) -> 0603; Website (none) -> https://www.digikey.pt/pt/products/detail/stackpole-electro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
- R22, R27: Manufacturer_Name (none) -> Stackpole Electronics Inc; Manufacturer_Part_Number (none) -> RNCF0603DTE100K; Package/Footprint (none) -> 0603; Website (none) -> https://www.digikey.pt/pt/products/detail/stackpole-electro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
- R23, R24, R28, R29: Manufacturer_Name (none) -> Stackpole Electronics Inc; Manufacturer_Part_Number (none) -> RNCF0603BTE10K0; Package/Footprint (none) -> 0603; Website (none) -> https://www.digikey.pt/pt/products/detail/stackpole-electro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
- R25, R30: Manufacturer_Name (none) -> Stackpole Electronics Inc; Manufacturer_Part_Number (none) -> RMCF0603FT200K; Package/Footprint (none) -> 0603; Website (none) -> https://www.digikey.pt/pt/products/detail/stackpole-electro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
