File: 2.Satellite/1.Hardware/Boards/avionics-batteryboard/batteryboard-bottom/batteryboard-bottom.kicad_sch (KiCad schematic)
At the start: 9 parts, among them J1 SFC-110-T2-X-D-A, J2 FTS-107-01-X-DV-A, U1 INA219BxD

Commit message: update BOM
Parts:
- C3: Manufacturer_Name (none) -> KYOCERA AVX; Manufacturer_Part_Number (none) -> 06035C104K4T2A; Package/Footprint (none) -> 0603; Website (none) -> https://www.digikey.pt/pt/products/detail/kyocera-avx/KAM15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
- J1: LCSC Part# C3323528 -> (none); Manufacturer_Name (none) -> Samtec Inc.; Package/Footprint (none) -> -
- J2: Manufacturer_Name (none) -> Samtec Inc.; Package/Footprint (none) -> -
- R1: Manufacturer_Name (none) -> Stackpole Electronics Inc; Manufacturer_Part_Number (none) -> CSM2512FT40L0; Package/Footprint (none) -> 2512; Website (none) -> https://www.digikey.pt/pt/products/detail/stackpole-electro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
- U1: LCSC Part# C2155799 -> (none); Manufacturer_Name (none) -> Texas Instruments; Package/Footprint (none) -> 8-SOIC
Changed lines of the file:
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@@
       (effects (font (size 1.27 1.27)) hide)
     )
-    (property "Datasheet" "http://www.ti.com/lit/ds/symlink/ina219.pdf" (at 67.691 55.118 0)
-      (effects (font (size 1.27 1.27)) hide)
-    )
-    (property "LCSC Part#" "C2155799" (at 58.801 52.578 0)
+    (property "Datasheet" "" (at 67.691 55.118 0)
       (effects (font (size 1.27 1.27)) hide)
     )
@@
     )
     (property "Website" "https://www.digikey.pt/pt/products/detail/texas-instruments/INA219BIDR/2426057?s=N4IgTCBcDaIJIDkCCYCMBOAQnAIgJRAF0BfIA" (at 58.801 52.578 0)
+      (effects (font (size 1.27 1.27)) hide)
+    )
+    (property "Description" "IC CURRENT MONITOR 0.5% 8SOIC" (at 58.801 52.578 0)
+      (effects (font (size 1.27 1.27)) hide)
+    )
+    (property "Manufacturer_Name" "Texas Instruments" (at 58.801 52.578 0)
+      (effects (font (size 1.27 1.27)) hide)
+    )
+    (property "Package/Footprint" "8-SOIC" (at 58.801 52.578 0)
       (effects (font (size 1.27 1.27)) hide)
     )
@@
       (effects (font (size 1.27 1.27)) hide)
     )
-    (property "Datasheet" "~" (at 40.386 52.578 0)
-      (effects (font (size 1.27 1.27)) hide)
-    )
-    (property "LCSC Part#" "" (at 40.386 52.578 0)
-      (effects (font (size 1.27 1.27)) hide)
-    )
-    (property "Website" "" (at 40.386 52.578 0)
+    (property "Datasheet" "" (at 40.386 52.578 0)
+      (effects (font (size 1.27 1.27)) hide)
+    )
+    (property "Website" "https://www.digikey.pt/pt/products/detail/stackpole-electronics-inc/CSM2512FT40L0/13930213?s=N4IgTCBcDaIMIGUCyYCsBGMAxAKgFgAYAZAkAXQF8g" (at 40.386 52.578 0)
+      (effects (font (size 1.27 1.27)) hide)
+    )
+    (property "Description" "RES 0.04 OHM 1% 3W 2512" (at 40.386 52.578 0)
+      (effects (font (size 1.27 1.27)) hide)
+    )
+    (property "Manufacturer_Name" "Stackpole Electronics Inc" (at 40.386 52.578 0)
+      (effects (font (size 1.27 1.27)) hide)
+    )
+    (property "Manufacturer_Part_Number" "CSM2512FT40L0" (at 40.386 52.578 0)
+      (effects (font (size 1.27 1.27)) hide)
+    )
+    (property "Package/Footprint" "2512" (at 40.386 52.578 0)
       (effects (font (size 1.27 1.27)) hide)
     )
@@
       (effects (font (size 1.27 1.27)) hide)
     )
-    (property "Datasheet" "~" (at 38.354 123.317 0)
-      (effects (font (size 1.27 1.27)) hide)
-    )
-    (property "LCSC Part#" "" (at 38.354 123.317 0)
+    (property "Datasheet" "" (at 38.354 123.317 0)
       (effects (font (size 1.27 1.27)) hide)
     )
@@
       (effects (font (size 1.27 1.27)) hide)
     )
+    (property "Package/Footprint" "" (at 38.354 123.317 0)
+      (effects (font (size 1.27 1.27)) hide)
+    )
     (pin "1")
     (instances
@@
       (effects (font (size 1.27 1.27)) hide)
     )
-    (property "Datasheet" "~" (at 147.828 39.751 0)
-      (effects (font (size 1.27 1.27)) hide)
-    )
-    (property "LCSC Part#" "" (at 147.828 39.751 0)
+    (property "Datasheet" "" (at 147.828 39.751 0)
       (effects (font (size 1.27 1.27)) hide)
     )
@@
     )
     (property "Website" "https://www.digikey.pt/pt/products/detail/samtec-inc/FTS-107-01-L-DV-A/7343465" (at 147.828 39.751 0)
+      (effects (font (size 1.27 1.27)) hide)
+    )
+    (property "Description" "CONN HEADER SMD 14POS 1.27MM" (at 147.828 39.751 0)
+      (effects (font (size 1.27 1.27)) hide)
+    )
+    (property "Manufacturer_Name" "Samtec Inc." (at 147.828 39.751 0)
+      (effects (font (size 1.27 1.27)) hide)
+    )
+    (property "Package/Footprint" "-" (at 147.828 39.751 0)
       (effects (font (size 1.27 1.27)) hide)
     )
@@
       (effects (font (size 1.27 1.27)) hide)
     )
-    (property "Datasheet" "~" (at 147.828 78.74 0)
-      (effects (font (size 1.27 1.27)) hide)
-    )
-    (property "LCSC Part#" "C3323528" (at 147.828 78.74 0)
+    (property "Datasheet" "" (at 147.828 78.74 0)
       (effects (font (size 1.27 1.27)) hide)
     )
@@
     )
     (property "Website" "https://www.digikey.pt/pt/products/detail/samtec-inc/SFC-110-T2-F-D-A/6678600" (at 147.828 78.74 0)
+      (effects (font (size 1.27 1.27)) hide)
+    )
+    (property "Description" "CONN RCPT 20POS 0.05 GOLD SMD" (at 147.828 78.74 0)
+      (effects (font (size 1.27 1.27)) hide)
+    )
+    (property "Manufacturer_Name" "Samtec Inc." (at 147.828 78.74 0)
+      (effects (font (size 1.27 1.27)) hide)
+    )
+    (property "Package/Footprint" "-" (at 147.828 78.74 0)
       (effects (font (size 1.27 1.27)) hide)
     )
@@
       (effects (font (size 1.27 1.27)) hide)
     )
-    (property "Datasheet" "~" (at 56.007 117.983 0)
-      (effects (font (size 1.27 1.27)) hide)
-    )
-    (property "LCSC Part#" "" (at 56.007 117.983 0)
+    (property "Datasheet" "" (at 56.007 117.983 0)
       (effects (font (size 1.27 1.27)) hide)
     )
     (property "Website" "" (at 56.007 117.983 0)
+      (effects (font (size 1.27 1.27)) hide)
+    )
+    (property "Package/Footprint" "" (at 56.007 117.983 0)
       (effects (font (size 1.27 1.27)) hide)
     )
@@
       (effects (font (size 1.27 1.27)) hide)
     )
-    (property "Datasheet" "~" (at 56.007 123.444 0)
-      (effects (font (size 1.27 1.27)) hide)
-    )
-    (property "LCSC Part#" "" (at 56.007 123.444 0)
+    (property "Datasheet" "" (at 56.007 123.444 0)
       (effects (font (size 1.27 1.27)) hide)
     )
@@
       (effects (font (size 1.27 1.27)) hide)
     )
+    (property "Package/Footprint" "" (at 56.007 123.444 0)
+      (effects (font (size 1.27 1.27)) hide)
+    )
     (pin "1")
     (instances
@@
       (effects (font (size 1.27 1.27)) hide)
     )
-    (property "Datasheet" "~" (at 64.135 40.64 0)
-      (effects (font (size 1.27 1.27)) hide)
-    )
-    (property "LCSC Part#" "" (at 64.135 40.64 0)
-      (effects (font (size 1.27 1.27)) hide)
-    )
-    (property "Website" "" (at 64.135 40.64 0)
+    (property "Datasheet" "" (at 64.135 40.64 0)
+      (effects (font (size 1.27 1.27)) hide)
+    )
+    (property "Website" "https://www.digikey.pt/pt/products/detail/kyocera-avx/KAM15AR71H104KT/1950904?s=N4IgTCBcDaIAwDY4GYCsBhAjHALAaRwBUwBBEAXQF8g" (at 64.135 40.64 0)
+      (effects (font (size 1.27 1.27)) hide)
+    )
+    (property "Description" "CAP CER 0.1UF 50V X7R 0603" (at 64.135 40.64 0)
+      (effects (font (size 1.27 1.27)) hide)
+    )
+    (property "Manufacturer_Name" "KYOCERA AVX" (at 64.135 40.64 0)
+      (effects (font (size 1.27 1.27)) hide)
+    )
+    (property "Manufacturer_Part_Number" "06035C104K4T2A" (at 64.135 40.64 0)
+      (effects (font (size 1.27 1.27)) hide)
+    )
+    (property "Package/Footprint" "0603" (at 64.135 40.64 0)
       (effects (font (size 1.27 1.27)) hide)
     )
@@
       (effects (font (size 1.27 1.27)) hide)
     )
-    (property "Datasheet" "~" (at 38.481 117.983 0)
-      (effects (font (size 1.27 1.27)) hide)
-    )
-    (property "LCSC Part#" "" (at 38.481 117.983 0)
+    (property "Datasheet" "" (at 38.481 117.983 0)
       (effects (font (size 1.27 1.27)) hide)
     )
@@
       (effects (font (size 1.27 1.27)) hide)
     )
+    (property "Package/Footprint" "" (at 38.481 117.983 0)
+      (effects (font (size 1.27 1.27)) hide)
+    )
