File: 2.Satellite/1.Hardware/Boards/avionics-batteryboard/batteryboard-middle/batteryboard-middle.kicad_pcb (KiCad board)
At the start: 2 copper layers, 45.6 x 45.6 mm, 15 parts, among them J1 FLE-107-01-X-DV-A, J2 FTS-107-01-X-DV-A, J3 Battery Pads, J4 Battery Pads

Commit message: update BOM
Changed lines of the file:
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@@
     (property "ki_description" "Generic connector, double row, 02x07, odd/even pin numbering scheme (row 1 odd numbers, row 2 even numbers), script generated (kicad-library-utils/schlib/autogen/connector/)")
     (property "ki_keywords" "connector")
-    (fp_text reference "J2" (at 0 -5.334 90) (layer "F.SilkS") hide
+    (fp_text reference "J2" (at 0 -5.334 90) (layer "F.SilkS")
         (effects (font (size 1.5 1.5) (thickness 0.15)))
     )
@@
     (property "ki_description" "Generic connector, double row, 02x07, odd/even pin numbering scheme (row 1 odd numbers, row 2 even numbers), script generated (kicad-library-utils/schlib/autogen/connector/)")
     (property "ki_keywords" "connector")
-    (fp_text reference "J1" (at 0 3.429 90) (layer "B.SilkS") hide
+    (fp_text reference "J1" (at 0 3.429 90) (layer "B.SilkS")
         (effects (font (size 0.635 0.635) (thickness 0.1016)) (justify mirror))
     )
