File: 2.Satellite/1.Hardware/Boards/avionics-batteryboard/batteryboard-middle/batteryboard-middle.kicad_sch (KiCad schematic)
At the start: 8 parts, among them J1 FLE-107-01-X-DV-A, J2 FTS-107-01-X-DV-A, J3 Battery Pads, J4 Battery Pads

Commit message: update BOM
Parts:
- J1: Manufacturer_Name (none) -> Samtec Inc.; Manufacturer_Part_Number (none) -> FLE-107-01-G-DV-A; Website (none) -> https://www.digikey.pt/pt/products/detail/samtec-inc/FLE-10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
- J2: Manufacturer_Name (none) -> Samtec Inc.; Manufacturer_Part_Number (none) -> FTS-107-01-L-DV-A; Website (none) -> https://www.digikey.pt/pt/products/detail/samtec-inc/FTS-10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
Changed lines of the file:
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@@
+      (effects (font (size 1.27 1.27)) hide)
+    )
+    (property "DNI" "" (at 98.552 91.567 0)
+      (effects (font (size 1.27 1.27)) hide)
+    )
+    (property "Description" "" (at 98.552 91.567 0)
+      (effects (font (size 1.27 1.27)) hide)
+    )
+    (property "Manufacturer_Name" "" (at 98.552 91.567 0)
+      (effects (font (size 1.27 1.27)) hide)
+    )
+    (property "Manufacturer_Part_Number" "" (at 98.552 91.567 0)
+      (effects (font (size 1.27 1.27)) hide)
+    )
+    (property "Package/Footprint" "" (at 98.552 91.567 0)
+      (effects (font (size 1.27 1.27)) hide)
+    )
+    (property "Website" "" (at 98.552 91.567 0)
       (effects (font (size 1.27 1.27)) hide)
     )
@@
       (effects (font (size 1.27 1.27)) hide)
     )
+    (property "DNI" "" (at 116.205 86.233 0)
+      (effects (font (size 1.27 1.27)) hide)
+    )
+    (property "Description" "" (at 116.205 86.233 0)
+      (effects (font (size 1.27 1.27)) hide)
+    )
+    (property "Manufacturer_Name" "" (at 116.205 86.233 0)
+      (effects (font (size 1.27 1.27)) hide)
+    )
+    (property "Manufacturer_Part_Number" "" (at 116.205 86.233 0)
+      (effects (font (size 1.27 1.27)) hide)
+    )
+    (property "Package/Footprint" "" (at 116.205 86.233 0)
+      (effects (font (size 1.27 1.27)) hide)
+    )
+    (property "Website" "" (at 116.205 86.233 0)
+      (effects (font (size 1.27 1.27)) hide)
+    )
     (pin "1")
     (instances
@@
       (effects (font (size 1.27 1.27)) hide)
     )
+    (property "DNI" "" (at 116.205 91.694 0)
+      (effects (font (size 1.27 1.27)) hide)
+    )
+    (property "Description" "" (at 116.205 91.694 0)
+      (effects (font (size 1.27 1.27)) hide)
+    )
+    (property "Manufacturer_Name" "" (at 116.205 91.694 0)
+      (effects (font (size 1.27 1.27)) hide)
+    )
+    (property "Manufacturer_Part_Number" "" (at 116.205 91.694 0)
+      (effects (font (size 1.27 1.27)) hide)
+    )
+    (property "Package/Footprint" "" (at 116.205 91.694 0)
+      (effects (font (size 1.27 1.27)) hide)
+    )
+    (property "Website" "" (at 116.205 91.694 0)
+      (effects (font (size 1.27 1.27)) hide)
+    )
     (pin "1")
     (instances
@@
     )
     (property "Datasheet" "~" (at 98.679 86.233 0)
+      (effects (font (size 1.27 1.27)) hide)
+    )
+    (property "DNI" "" (at 98.679 86.233 0)
+      (effects (font (size 1.27 1.27)) hide)
+    )
+    (property "Description" "" (at 98.679 86.233 0)
+      (effects (font (size 1.27 1.27)) hide)
+    )
+    (property "Manufacturer_Name" "" (at 98.679 86.233 0)
+      (effects (font (size 1.27 1.27)) hide)
+    )
+    (property "Manufacturer_Part_Number" "" (at 98.679 86.233 0)
+      (effects (font (size 1.27 1.27)) hide)
+    )
+    (property "Package/Footprint" "" (at 98.679 86.233 0)
+      (effects (font (size 1.27 1.27)) hide)
+    )
+    (property "Website" "" (at 98.679 86.233 0)
       (effects (font (size 1.27 1.27)) hide)
     )
@@
       (effects (font (size 1.27 1.27)) hide)
     )
+    (property "DNI" "" (at 43.18 111.76 0)
+      (effects (font (size 1.27 1.27)) hide)
+    )
+    (property "Description" "" (at 43.18 111.76 0)
+      (effects (font (size 1.27 1.27)) hide)
+    )
+    (property "Manufacturer_Name" "" (at 43.18 111.76 0)
+      (effects (font (size 1.27 1.27)) hide)
+    )
+    (property "Manufacturer_Part_Number" "" (at 43.18 111.76 0)
+      (effects (font (size 1.27 1.27)) hide)
+    )
+    (property "Package/Footprint" "" (at 43.18 111.76 0)
+      (effects (font (size 1.27 1.27)) hide)
+    )
+    (property "Website" "" (at 43.18 111.76 0)
+      (effects (font (size 1.27 1.27)) hide)
+    )
     (pin "1")
     (pin "2")
@@
     )
     (property "Datasheet" "~" (at 59.182 58.928 0)
+      (effects (font (size 1.27 1.27)) hide)
+    )
+    (property "DNI" "" (at 59.182 58.928 0)
+      (effects (font (size 1.27 1.27)) hide)
+    )
+    (property "Description" "CONN RCPT 14POS 0.05 GOLD SMD" (at 59.182 58.928 0)
+      (effects (font (size 1.27 1.27)) hide)
+    )
+    (property "Manufacturer_Name" "Samtec Inc." (at 59.182 58.928 0)
+      (effects (font (size 1.27 1.27)) hide)
+    )
+    (property "Manufacturer_Part_Number" "FLE-107-01-G-DV-A" (at 59.182 58.928 0)
+      (effects (font (size 1.27 1.27)) hide)
+    )
+    (property "Package/Footprint" "" (at 59.182 58.928 0)
+      (effects (font (size 1.27 1.27)) hide)
+    )
+    (property "Website" "https://www.digikey.pt/pt/products/detail/samtec-inc/FLE-107-01-G-DV-A/6678142" (at 59.182 58.928 0)
       (effects (font (size 1.27 1.27)) hide)
     )
@@
       (effects (font (size 1.27 1.27)) hide)
     )
+    (property "DNI" "" (at 151.765 58.674 0)
+      (effects (font (size 1.27 1.27)) hide)
+    )
+    (property "Description" "CONN HEADER SMD 14POS 1.27MM" (at 151.765 58.674 0)
+      (effects (font (size 1.27 1.27)) hide)
+    )
+    (property "Manufacturer_Name" "Samtec Inc." (at 151.765 58.674 0)
+      (effects (font (size 1.27 1.27)) hide)
+    )
+    (property "Manufacturer_Part_Number" "FTS-107-01-L-DV-A" (at 151.765 58.674 0)
+      (effects (font (size 1.27 1.27)) hide)
+    )
+    (property "Package/Footprint" "" (at 151.765 58.674 0)
+      (effects (font (size 1.27 1.27)) hide)
+    )
+    (property "Website" "https://www.digikey.pt/pt/products/detail/samtec-inc/FTS-107-01-L-DV-A/7343465" (at 151.765 58.674 0)
+      (effects (font (size 1.27 1.27)) hide)
+    )
     (pin "1")
     (pin "10")
@@
       (effects (font (size 1.27 1.27)) hide)
     )
+    (property "DNI" "" (at 42.926 126.873 0)
+      (effects (font (size 1.27 1.27)) hide)
+    )
+    (property "Description" "" (at 42.926 126.873 0)
+      (effects (font (size 1.27 1.27)) hide)
+    )
+    (property "Manufacturer_Name" "" (at 42.926 126.873 0)
+      (effects (font (size 1.27 1.27)) hide)
+    )
+    (property "Manufacturer_Part_Number" "" (at 42.926 126.873 0)
+      (effects (font (size 1.27 1.27)) hide)
+    )
+    (property "Package/Footprint" "" (at 42.926 126.873 0)
+      (effects (font (size 1.27 1.27)) hide)
+    )
+    (property "Website" "" (at 42.926 126.873 0)
+      (effects (font (size 1.27 1.27)) hide)
+    )
