File: 2.Satellite/1.Hardware/Boards/avionics-batteryboard/batteryboard-top/batteryboard-top.kicad_sch (KiCad schematic)
At the start: 6 parts, among them J1 FLE-107-01-X-DV-A, J2 FLE-105-01-X-DV-A

Commit message: update BOM
Parts:
- J1: Manufacturer_Name (none) -> Samtec Inc.; Manufacturer_Part_Number (none) -> FLE-107-01-G-DV-A; Website (none) -> https://www.digikey.pt/pt/products/category/conectores-reta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
- J2: Manufacturer_Name (none) -> Samtec Inc.; Manufacturer_Part_Number (none) -> FLE-105-01-G-DV-A; Website (none) -> https://www.digikey.pt/pt/products/detail/samtec-inc/FLE-10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
Changed lines of the file:
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@@
+      (effects (font (size 1.27 1.27)) hide)
+    )
+    (property "DNI" "" (at 96.266 93.599 0)
+      (effects (font (size 1.27 1.27)) hide)
+    )
+    (property "Description" "" (at 96.266 93.599 0)
+      (effects (font (size 1.27 1.27)) hide)
+    )
+    (property "Manufacturer_Name" "" (at 96.266 93.599 0)
+      (effects (font (size 1.27 1.27)) hide)
+    )
+    (property "Manufacturer_Part_Number" "" (at 96.266 93.599 0)
+      (effects (font (size 1.27 1.27)) hide)
+    )
+    (property "Package/Footprint" "" (at 96.266 93.599 0)
+      (effects (font (size 1.27 1.27)) hide)
+    )
+    (property "Website" "" (at 96.266 93.599 0)
       (effects (font (size 1.27 1.27)) hide)
     )
@@
       (effects (font (size 1.27 1.27)) hide)
     )
+    (property "DNI" "" (at 113.919 88.265 0)
+      (effects (font (size 1.27 1.27)) hide)
+    )
+    (property "Description" "" (at 113.919 88.265 0)
+      (effects (font (size 1.27 1.27)) hide)
+    )
+    (property "Manufacturer_Name" "" (at 113.919 88.265 0)
+      (effects (font (size 1.27 1.27)) hide)
+    )
+    (property "Manufacturer_Part_Number" "" (at 113.919 88.265 0)
+      (effects (font (size 1.27 1.27)) hide)
+    )
+    (property "Package/Footprint" "" (at 113.919 88.265 0)
+      (effects (font (size 1.27 1.27)) hide)
+    )
+    (property "Website" "" (at 113.919 88.265 0)
+      (effects (font (size 1.27 1.27)) hide)
+    )
     (pin "1")
     (instances
@@
     )
     (property "Datasheet" "~" (at 61.595 57.023 0)
+      (effects (font (size 1.27 1.27)) hide)
+    )
+    (property "DNI" "" (at 61.595 57.023 0)
+      (effects (font (size 1.27 1.27)) hide)
+    )
+    (property "Description" "CONN RCPT 14POS 0.05 GOLD SMD" (at 61.595 57.023 0)
+      (effects (font (size 1.27 1.27)) hide)
+    )
+    (property "Manufacturer_Name" "Samtec Inc." (at 61.595 57.023 0)
+      (effects (font (size 1.27 1.27)) hide)
+    )
+    (property "Manufacturer_Part_Number" "FLE-107-01-G-DV-A" (at 61.595 57.023 0)
+      (effects (font (size 1.27 1.27)) hide)
+    )
+    (property "Package/Footprint" "" (at 61.595 57.023 0)
+      (effects (font (size 1.27 1.27)) hide)
+    )
+    (property "Website" "https://www.digikey.pt/pt/products/category/conectores-retangulares/2027?s=N4IgTCBcDaIGIBkCiBaAjABgOwo2lA4igCIBqKAgiALoC%20QA" (at 61.595 57.023 0)
       (effects (font (size 1.27 1.27)) hide)
     )
@@
       (effects (font (size 1.27 1.27)) hide)
     )
+    (property "DNI" "" (at 113.919 93.726 0)
+      (effects (font (size 1.27 1.27)) hide)
+    )
+    (property "Description" "" (at 113.919 93.726 0)
+      (effects (font (size 1.27 1.27)) hide)
+    )
+    (property "Manufacturer_Name" "" (at 113.919 93.726 0)
+      (effects (font (size 1.27 1.27)) hide)
+    )
+    (property "Manufacturer_Part_Number" "" (at 113.919 93.726 0)
+      (effects (font (size 1.27 1.27)) hide)
+    )
+    (property "Package/Footprint" "" (at 113.919 93.726 0)
+      (effects (font (size 1.27 1.27)) hide)
+    )
+    (property "Website" "" (at 113.919 93.726 0)
+      (effects (font (size 1.27 1.27)) hide)
+    )
     (pin "1")
     (instances
@@
       (effects (font (size 1.27 1.27)) hide)
     )
+    (property "DNI" "" (at 96.393 88.265 0)
+      (effects (font (size 1.27 1.27)) hide)
+    )
+    (property "Description" "" (at 96.393 88.265 0)
+      (effects (font (size 1.27 1.27)) hide)
+    )
+    (property "Manufacturer_Name" "" (at 96.393 88.265 0)
+      (effects (font (size 1.27 1.27)) hide)
+    )
+    (property "Manufacturer_Part_Number" "" (at 96.393 88.265 0)
+      (effects (font (size 1.27 1.27)) hide)
+    )
+    (property "Package/Footprint" "" (at 96.393 88.265 0)
+      (effects (font (size 1.27 1.27)) hide)
+    )
+    (property "Website" "" (at 96.393 88.265 0)
+      (effects (font (size 1.27 1.27)) hide)
+    )
     (pin "1")
     (instances
@@
       (effects (font (size 1.27 1.27)) hide)
     )
+    (property "DNI" "" (at 157.734 54.991 0)
+      (effects (font (size 1.27 1.27)) hide)
+    )
+    (property "Description" "CONN RCPT 10POS 0.05 GOLD SMD" (at 157.734 54.991 0)
+      (effects (font (size 1.27 1.27)) hide)
+    )
+    (property "Manufacturer_Name" "Samtec Inc." (at 157.734 54.991 0)
+      (effects (font (size 1.27 1.27)) hide)
+    )
+    (property "Manufacturer_Part_Number" "FLE-105-01-G-DV-A" (at 157.734 54.991 0)
+      (effects (font (size 1.27 1.27)) hide)
+    )
+    (property "Package/Footprint" "" (at 157.734 54.991 0)
+      (effects (font (size 1.27 1.27)) hide)
+    )
+    (property "Website" "https://www.digikey.pt/pt/products/detail/samtec-inc/FLE-105-01-G-DV-A/2651128" (at 157.734 54.991 0)
+      (effects (font (size 1.27 1.27)) hide)
+    )
